Commit message: Added hider bot

File: urdf/turtlebot3_waffle_pi_hider.urdf.xacro (robot description, xacro)
@@ -136,5 +136,5 @@
     <parent link="base_link"/>
     <child link="base_scan"/>
-    <origin xyz="-0.064 0 0.122" rpy="0 0 0"/>
+    <origin xyz="-0.064 0 0.244" rpy="0 0 0"/>
   </joint>
   <link name="base_scan">
