Commit message: WIP: pursuit

File: urdf/turtlebot3_waffle_pi_seeker.gazebo.xacro (robot description, xacro)
@@ -5,5 +5,5 @@
   <xacro:arg name="imu_visual"    default="false"/>
   <gazebo reference="base_link">
-    <material>Gazebo/Red </material>
+    <material>Gazebo/Blue </material>
   </gazebo>
   <gazebo reference="wheel_left_link">
